Commit message: Corrections of camera links and parents

File: catkin_ws_project4/src/my_robot/urdf/my_robot.xacro (robot description, xacro)
@@ -118,5 +118,4 @@
     <dynamics damping="1.0" friction="1.0"/>
   </joint>
-  <!--
   <link name='camera'>
     <visual name='camera_visual'>
@@ -148,8 +147,7 @@
     <axis xyz="0 1 0" rpy="0 0 0"/>
   </joint>
-  -->
   <joint name="camera_optical_joint" type="fixed">
-    <origin xyz=".2 0 0" rpy="0 0 0"/>
-    <parent link="chassis"/>
+    <origin xyz="0 0 0" rpy="-1.5707 0 -1.5707"/>
+    <parent link="camera"/>
     <child link="camera_link_optical"/>
   </joint>
